File: MainPCB/EnvMCRO.sch (KiCad schematic (older format))
At the start: 29 parts, among them U1 Pico

Commit message: Added Pads/traces for 3535 SK6812 or WS2812B
Parts:
- added D1, D10, D11, D12, D2, D3, D4, D5, D6, D7, D8, D9: SK6812, LED_SMD:LED_SK6812MINI_PLCC4_3.5x3.5mm_P1.75mm, symbol LED:SK6812
Connections:
- net GND: now also D1.1 (VSS), D10.1 (VSS), D11.1 (VSS), D12.1 (VSS), D2.1 (VSS), D3.1 (VSS), D4.1 (VSS), D5.1 (VSS), D6.1 (VSS), D7.1 (VSS), D8.1 (VSS), D9.1 (VSS)
- net VBUS: now reaches U1.40 (VBUS)
- net VBUS: now also D1.3 (VDD), D10.3 (VDD), D11.3 (VDD), D12.3 (VDD), D2.3 (VDD), D3.3 (VDD), D4.3 (VDD), D5.3 (VDD), D6.3 (VDD), D7.3 (VDD), D8.3 (VDD), D9.3 (VDD)
- net LEDDINPIN: now reaches U1.7 (GPIO5)
- net LEDDINPIN: now also D1.2 (DIN)
- new net: D1.4 (DOUT), D2.2 (DIN)
- new net: D2.4 (DOUT), D3.2 (DIN)
- new net: D3.4 (DOUT), D4.2 (DIN)
- new net: D4.4 (DOUT), D5.2 (DIN)
- new net: D5.4 (DOUT), D6.2 (DIN)
- new net: D6.4 (DOUT), D7.2 (DIN)
- new net: D7.4 (DOUT), D8.2 (DIN)
- new net: D8.4 (DOUT), D9.2 (DIN)
- new net: D10.2 (DIN), D9.4 (DOUT)
- new net: D10.4 (DOUT), D11.2 (DIN)
- new net: D11.4 (DOUT), D12.2 (DIN)

Commit message: better RGB implementation using SK6812 MINI E footprints to be installed reverse on the back of the PCB + generated gerber
Parts:
- removed D1, D10, D11, D12, D2, D3, D4, D5, D6, D7, D8, D9: SK6812, LED_SMD:LED_SK6812MINI_PLCC4_3.5x3.5mm_P1.75mm, symbol LED:SK6812
- added D1, D10, D11, D12, D2, D3, D4, D5, D6, D7, D8, D9: SK6812MINI-E, sk6812mini:MX_SK6812MINI-E_REV, symbol kicad-keyboard-parts:SK6812MINI-E
Connections:
- net GND: now also D1.3 (VSS), D10.3 (VSS), D11.3 (VSS), D12.3 (VSS), D2.3 (VSS), D3.3 (VSS), D4.3 (VSS), D5.3 (VSS), D6.3 (VSS), D7.3 (VSS), D8.3 (VSS), D9.3 (VSS)
- net LEDDINPIN: now also U1.1 (GPIO0), D1.4 (DIN); no longer U1.7 (GPIO5)
- net VBUS: now also D1.1 (VDD), D10.1 (VDD), D11.1 (VDD), D12.1 (VDD), D2.1 (VDD), D3.1 (VDD), D4.1 (VDD), D5.1 (VDD), D6.1 (VDD), D7.1 (VDD), D8.1 (VDD), D9.1 (VDD)
- new net: D1.2 (DOUT), D2.4 (DIN)
- new net: D2.2 (DOUT), D3.4 (DIN)
- new net: D3.2 (DOUT), D4.4 (DIN)
- new net: D4.2 (DOUT), D5.4 (DIN)
- new net: D5.2 (DOUT), D6.4 (DIN)
- new net: D6.2 (DOUT), D7.4 (DIN)
- new net: D7.2 (DOUT), D8.4 (DIN)
- new net: D8.2 (DOUT), D9.4 (DIN)
- new net: D10.4 (DIN), D9.2 (DOUT)
- new net: D10.2 (DOUT), D11.4 (DIN)
- new net: D11.2 (DOUT), D12.4 (DIN)
