File: MainPCB_RPI-PICO/EnvMCRO.sch (KiCad schematic (older format))
At the start: 47 parts, among them SW1 Rotary_Encoder_Switch, U1 Pico

Commit message: updated macro boards to have padded mount holes and github url
Parts:
- removed K_12, K_13: KEYSW, Connector_PinHeader_2.54mm:PinHeader_1x02_P2.54mm_Vertical, symbol MX_Alps_Hybrid:MX-NoLED
- added SW2, SW3: Rotary_Encoder_Switch, Rotary_Encoder:RotaryEncoder_Alps_EC11E-Switch_Vertical_H20mm, symbol Device:Rotary_Encoder_Switch
- H1, H2, H3, H4: footprint MountingHole:MountingHole_2.2mm_M2 -> MountingHole:MountingHole_2.2mm_M2_Pad; symbol Mechanical:MountingHole -> Mechanical:MountingHole_Pad
Connections:
- net GND: now also H1.1, H2.1, H3.1, H4.1, SW2.C, SW3.C
- net ROTA: now also SW1.B, SW2.B, SW3.B; no longer SW1.A
- net ROTB: now also SW1.A, SW2.A, SW3.A; no longer SW1.B
- net col4: now also SW1.S2, SW2.S2, SW3.S2; no longer SW1.S1
- net at D_14.2 (A): now also SW1.S1; no longer SW1.S2
- net at D_13.2 (A): now also SW3.S1
- net at D_12.2 (A): now also SW2.S1
Other:
- moved on the sheet: D1, D10, D11, D12, D2, D3, D4, D5, D6, D7, D8, D9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

Commit message: swapped EC11 for EC12 because cheaper, might swap again to what ever people get a hold of the easiest.
Parts:
- SW1, SW2, SW3: footprint Rotary_Encoder:RotaryEncoder_Alps_EC11E-Switch_Vertical_H20mm -> Rotary_Encoder:RotaryEncoder_Alps_EC12E-Switch_Vertical_H20mm
Changed lines of the file:
@@
 F 0 "SW1" H 5400 3000 50  0000 C CNN
 F 1 "Rotary_Encoder_Switch" H 5400 3026 50  0001 C CNN
-F 2 "Rotary_Encoder:RotaryEncoder_Alps_EC11E-Switch_Vertical_H20mm" H 5250 2910 50  0001 C CNN
+F 2 "Rotary_Encoder:RotaryEncoder_Alps_EC12E-Switch_Vertical_H20mm" H 5250 2910 50  0001 C CNN
 F 3 "~" H 5400 3010 50  0001 C CNN
 	1    5400 2750
@@
 F 0 "SW3" H 5400 2150 50  0000 C CNN
 F 1 "Rotary_Encoder_Switch" H 5400 2176 50  0001 C CNN
-F 2 "Rotary_Encoder:RotaryEncoder_Alps_EC11E-Switch_Vertical_H20mm" H 5250 2060 50  0001 C CNN
+F 2 "Rotary_Encoder:RotaryEncoder_Alps_EC12E-Switch_Vertical_H20mm" H 5250 2060 50  0001 C CNN
 F 3 "~" H 5400 2160 50  0001 C CNN
 	1    5400 1900
@@
 F 0 "SW2" H 5400 1150 50  0000 C CNN
 F 1 "Rotary_Encoder_Switch" H 5400 1176 50  0001 C CNN
-F 2 "Rotary_Encoder:RotaryEncoder_Alps_EC11E-Switch_Vertical_H20mm" H 5250 1060 50  0001 C CNN
+F 2 "Rotary_Encoder:RotaryEncoder_Alps_EC12E-Switch_Vertical_H20mm" H 5250 1060 50  0001 C CNN
 F 3 "~" H 5400 1160 50  0001 C CNN
 	1    5400 900
